File: ins-board.sch (KiCad schematic (older format))
At the start: 76 parts, among them P1 PWR, P2 Power (Solder Pad), Q1 FDN306P, Q2 FDC638APZ, U1 24LC128, U2 STM32F415RGT6, U3 LTC4412, U4 MAX3051, U5 LT1965, U6 LT1761-3.3, U7 LT1965, X1 CRYSTAL 16MHz 10ppm

Commit message: rocket board
Parts:
- removed C13, C17: 0.1uF, symbol C
- removed C18, C22: 10uF, ~, symbol C
- removed C20, C23, C25: 10uF, symbol C
- removed C21, C27: 1uF, symbol C
- removed C24: 0.01uF, symbol C
- removed C26: 100uF, symbol C
- removed CONN1: JTAG, MODULE, symbol JTAG
- removed CONN6, CONN7, CONN8, CONN9: UART, MODULE, symbol UART
- removed D1: SD ACT, symbol LED
- removed D4: STATUS, symbol LED
- removed D6: BAS52-02V, symbol DIODESCH
- removed F1: FUSE 500mA, symbol FUSE
- removed FB1: BLM18KG601SN1, symbol FILTER
- removed P2: Power (Solder Pad), ~, symbol CONN_2
- removed Q1: FDN306P, symbol MOSFET_P
- removed Q2: FDC638APZ, symbol MOS_P
- removed R1, R8: 1k, symbol R
- removed R14, R21: 47k, ~, symbol R
- removed R2: 10k, symbol R
- removed R20: 47k, symbol R
- removed U1: 24LC128, MODULE, symbol 24LC128
- removed U3: LTC4412, MODULE, symbol LTC4412
- removed U5, U7: LT1965, MODULE, symbol LT1965
- removed U6: LT1761-3.3, MODULE, symbol LT1761-3.3
- added C?: C, symbol C
- added C?: 10nF, symbol C
- added C? (x6): 0.1uF, symbol C
- added C?: 2.2nF 50V, symbol C
- added C?: 0.22uF, symbol C
- added C?: 4.7uF, symbol C
- added C?: 10uF, ~, symbol C
- added CONN?: SWD, MODULE, symbol SWD
- added U?: MPU6000, MODULE, symbol MPU6000
- added U?: HMC5883L, MODULE, symbol HMC5883L
- added U?: MS5611-01BA, MODULE, symbol MS5611-01BA
- added U?: H3LIS331DL, MODULE, symbol H3LIS331DL
- R16, R17: value 4.7k -> DNP
- R5: value 10k -> 100k
Connections:
- net labels removed: V_IN
- wire segments 154 -> 143
- no-connect marks 5 -> 7
Other:
- note removed: "3.6V...20V"
- note removed: "502570-0893"
- note removed: "Address: 0xA0"
- note removed: "EEPROM"
- note removed: "SanDisk Ultra:\nr/w 150mA\nsleep 350uA"
- note removed: "ideal diode controller"
- note removed: "needed for ST USB-Bootloader"
- moved on the sheet: C1, C19, C3, CONN2, CONN3, CONN4, CONN5, D5, P1, R12, R13, R15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

Commit message: schematics
Parts:
- removed CONN3: MICRO_USB, symbol MICRO_USB
- removed CONN4: I2C/UART, MODULE, symbol I2C
- removed R12, R13: 22, symbol R
- removed R15: 0, symbol R
- removed R16, R17: DNP, symbol R
- added C? (x3): C, symbol C
- added CONN?: UART, MODULE, symbol UART
- added U?: MIC5201-3.3YS, symbol MIC5201-3.3YS
Connections:
- net VCC_A is gone; now on net VCC: C?.1, C?.1, C?.1, C?.1, C?.1, C?.1, R10.1, R11.1, U?.1 (VDD), U?.1 (Vdd_IO), U?.13 (VDD), U?.13 (VDDIO), U?.14 (Vdd), U?.15 (Rsvd_(Vdd)), U?.2 (PS), U?.2 (VDD), U?.4 (S1), U?.7 (SA0), U?.8 (CS)
- net VCC_IO is gone; now on net V_DC: CONN5.1 (VCC)
- net GND: now also U4.8 (RS), C?.2, C?.2, C?.2, CONN?.2 (GND), CONN?.MECH (GND), U?.2 (GND)
- net VCC: now also CONN?.1 (VCC), U?.3 (OUT)
- net V_DC: now also U?.1 (IN)
- no-connect marks 7 -> 5
Other:
- note removed: "RRS (kΩ)\n≈ 12000 / (maximum speed in kbps)"
- moved on the sheet: C19, C?, CONN5, P1, R18, U4, U?

Commit message: stm32f042
Parts:
- removed C11, C12: 2.2uF, symbol C
- removed U2: STM32F415RGT6, MODULE, symbol STM32F415RGT6
- added U?: STM32F042C6T6, MODULE, symbol STM32F042C6T6
Connections:
- net CAN_CONN1_RX: now also U?.25 (PB12)
- net CAN_CONN1_TX: now also U?.26 (PB13)
- net ERROR_LED: now also U?.31 (PA10)
- net GND: now also CONN?.2 (GND), U?.23 (VSS_2), U?.35 (VSS_3), U?.44 (BOOT0), U?.47 (VSS_1), U?.8 (VSSA)
- net HEARTBEAT_LED: now also U?.29 (PA8)
- net HMC5883L_DRDY: now also U?.18 (PB0)
- net I2C_CONN1_SCL: now also U?.21 (PB10)
- net I2C_CONN1_SDA: now also U?.22 (PB11)
- net INT_I2C_SCL: now also U?.45 (PB8)
- net INT_I2C_SDA: now also U?.46 (PB9)
- net MPU6000_INT: now also U?.4 (PC15/OSC32_OUT)
- net SD_DETECT: now also U?.3 (PC14/OSC32_IN)
- net SD_LED: now also U?.28 (PB15)
- net STATUS_LED: now also U?.27 (PB14)
- net STM32F4_NRST: now also CONN?.3 (NRST), U?.7 (NRST)
- net VCC: now also CONN?.1 (VCC), U?.1 (VBAT), U?.24 (VDD_2), U?.36 (VDDIO2), U?.48 (VDD_1), U?.9 (VDDA)
- net V_BAT_MON_AD: now also U?.2 (PC13)
- net V_USB: now also U?.30 (PA9)
- net at C16.1, X1.1: now also U?.6 (PF1/OSC_OUT)
- net at C15.1, X1.3: now also U?.5 (PF0/OSC_IN)
- no-connect marks 5 -> 4
Other:
- note removed: "(SPI3_MISO)"
- note removed: "(SPI3_MOSI)"
- note removed: "(SPI3_NSS)"
- note removed: "(SPI3_SCK)"
- note removed: "CAN2_RX"
- note removed: "CAN2_TX"
- note removed: "I2C1_SCL"
- note removed: "I2C1_SDA"
- note removed: "I2C2_SCL (UART3_TX)"
- note removed: "I2C2_SDA (UART3_RX)"
- note removed: "SPI1_MISO"
- note removed: "SPI1_MOSI"
- note removed: "SPI1_SCK"
- note removed: "UART1_RX"
- note removed: "UART1_TX"
- note removed: "UART2_RX"
- note removed: "UART2_TX"
- note removed: "UART4_RX"
- note removed: "UART4_TX"
- note removed: "UART6_RX"
- note removed: "UART6_TX"
- moved on the sheet: C15, C16, CONN?, X1

Commit message: Done
Parts:
- gave numbers to parts that had none: 23
- renumbered C2 to C1, C14 to C12, C15 to C13, C16 to C14, C19 to C16, C1 to C2, C4 to C3, C5 to C4, C3 to C5, CONN5 to CONN3, D2 to D1, D3 to D2, D5 to D3, R3 to R1, R4 to R2, R5 to R3, R6 to R4, R7 to R5, R9 to R6, R10 to R7, R11 to R8, R18 to R9, U4 to U3
Connections:
- net SD_LED is gone; now on net SDIO_DIN: U1.28 (PB15)
- net STATUS_LED is gone; now on net SD_DOUT: U1.27 (PB14)
- net V_USB is gone; now on net UART_TX: U1.30 (PA9)
- net CAN_CONN1_RX: now also U1.45 (PB8); no longer U1.25 (PB12)
- net CAN_CONN1_TX: now also U1.46 (PB9); no longer U1.26 (PB13)
- net ERROR_LED: now also U1.38 (PA15); no longer U1.31 (PA10)
- net H3LIS331DL_INT1: now also U1.19 (PB1)
- net INT_I2C_SCL: now also U1.42 (PB6); no longer U1.45 (PB8)
- net INT_I2C_SDA: now also U1.43 (PB7); no longer U1.46 (PB9)
- net MPU6000_INT: now also U1.20 (PB2); no longer U1.4 (PC15/OSC32_OUT)
- net SD_DETECT: now also U1.39 (PB3); no longer U1.3 (PC14/OSC32_IN)
- net V_BAT_MON_AD: now also U1.11 (PA1); no longer U1.2 (PC13)
- net STM32F4_SWDIO: now reaches CONN1.4 (SWDIO)
- net STM32F4_SWDIO: now also U1.34 (PA13)
- net STM32F4_SWCLK: now reaches CONN1.5 (SWCLK)
- net STM32F4_SWCLK: now also U1.37 (PA14)
- net UART_TX: now reaches CONN4.3 (TX)
- net UART_RX: now reaches CONN4.4 (RX)
- net UART_RX: now also U1.31 (PA10)
- net I2C_CONN1_SCL: no longer names the net of U1.21 (PB10)
- net I2C_CONN1_SDA: no longer names the net of U1.22 (PB11)
- net SDIO_CK renamed SDIO_CLK
- net SDIO_CLK: now also U1.26 (PB13)
- net SDIO_CMD renamed SDIO_DIN
- net SDIO_D0 renamed SD_DOUT
- net SDIO_D1: no longer names the net of CONN2.8 (DAT1)
- net SDIO_D2: no longer names the net of CONN2.1 (DAT2)
- net SDIO_D3: no longer names the net of CONN2.2 (DAT3)
- no-connect marks 4 -> 7
Other:
- note added: "MISO"
- note added: "MOSI"
- note added: "SCLK"
- moved on the sheet: R7, R8
