File: ins-board.kicad_pcb (KiCad board)
At the start: 4 copper layers, 50 x 23 mm, 94 parts, among them P1 PWR, P2 Power (Solder Pad), Q1 FDN306P, Q2 FDC638APZ, U1 24LC128, U10 HMC5883L, U11 H3LIS331DL, U2 STM32F415RGT6, U3 LTC4412, U4 MAX3051, U5 LT1965, U6 LT1761-3.3, U7 LT1965, U8 MS5611-01BA, U9 MPU6000, X1 CRYSTAL 16MHz 10ppm

Commit message: pcb + footprints
Parts:
- removed C22, C23, C25, C37: 10uF, _0603-W
- removed C24: 0.01uF, _0603-W
- removed C26: 100uF, SM1206
- removed C27: 1uF, _0603-W
- removed C28, C29, C30, C32, C33, C34: 0.1uF, _0603-W
- removed C31: 2.2nF 50V, _0603-W
- removed C35: 0.22uF, _0603-W
- removed C36: 4.7uF, _0603-W
- removed CONN4: I2C/UART, _Molex-PicoBlade-SMD-4
- removed CONN5: CAN, _Molex-PicoBlade-SMD-4
- removed CONN6, CONN7, CONN8, CONN9: UART, _Molex-PicoBlade-SMD-4
- removed D3: ERROR, _0603-W
- removed D4: STATUS, _0603-W
- removed D5: HEARTBEAT, _0603-W
- removed D6: BAS52-02V, _SC79
- removed F1: FUSE 500mA, _0603-W
- removed FB1: BLM18KG601SN1, _0603-W
- removed Q1: FDN306P, _FAIRCHILD-MOSFET-SuperSOT-3
- removed Q2: FDC638APZ, _FAIRCHILD-MOSFET-SuperSOT-6
- removed R14, R20, R21: 47k, _0603-W
- removed R15: 0, _0603-W
- removed R16, R17: 4.7k, _0603-W
- removed R18: NP / 120, _0603-W
- removed U10: HMC5883L, _HMC5883L
- removed U11: H3LIS331DL, _H3LIS331DL
- removed U6: LT1761-3.3, _TSOT23-5
- removed U7: LT1965, _MSOP-8-EP
- removed U8: MS5611-01BA, _MS5611-01BA
- removed U9: MPU6000, _MPU-60X0
- removed _M2 (x4): VAL**, _M2
- C1, C14, C3, C4, C6, C7, C8, C9, R5: footprint _0603-W -> _std:_0603-W
- C10: value 0.1uF -> 10pF; footprint _0603-W -> _std:_0603-W
- C11: value 2.2uF -> 10pF; footprint _0603-W -> _std:_0603-W
- C12: value 2.2uF -> 1uF; footprint _0603-W -> _std:_0603-W
- C13: value 0.1uF -> 10uF; footprint _0603-W -> _std:_0603-W; moved to F.Cu
- C15: value 10pF -> 0.1uF; footprint _0603-W -> _std:_0603-W
- C16: value 10pF -> 10uF; footprint _0603-W -> _std:_0603-W
- C17, R2: footprint _0603-W -> _std:_0603-W; moved to F.Cu
- C18: value 10uF -> 0.1uF; footprint _0603-W -> _std:_0603-W; moved to F.Cu
- C19: value 0.1uF -> 2.2nF 50V; footprint _0603-W -> _std:_0603-W; moved to F.Cu
- C2, C5: value 1uF -> 0.1uF; footprint _0603-W -> _std:_0603-W
- C20: value 10uF -> 0.1uF; footprint _0603-W -> _std:_0603-W
- C21: value 1uF -> 10nF; footprint _0603-W -> _std:_0603-W; moved to F.Cu
- CONN1: value JTAG -> SWD; footprint _Molex-PicoBlade-SMD-8 -> _connectors:_Pin2mm_5z
- CONN2: footprint _Molex-microSD-502570-0893 -> _div:_Molex-microSD-502570-0893; moved to F.Cu
- CONN3: value MICRO_USB -> UART; footprint _Micro-USB-AB-receptacle-SMT -> _connectors:_Molex-PicoBlade-SMD-4
- D1: value SD ACT -> ERROR; footprint _0603-W -> _std:_0603-W; moved to F.Cu
- D2: value POWER -> HEARTBEAT; footprint _0603-W -> _std:_0603-W; moved to F.Cu
- P1: value PWR -> CONN_8; footprint _Molex-PicoBlade-SMD-2 -> _connectors:_Solder_Pad1.27_8; moved to F.Cu
- P2: value Power (Solder Pad) -> PWR; footprint _Solder_Pad2.54_2 -> _connectors:_Molex-PicoBlade-SMD-2
- R1: value 1k -> 15k; footprint _0603-W -> _std:_0603-W; moved to F.Cu
- R10: value 4.7k -> 1k; footprint _0603-W -> _std:_0603-W
- R11: value 4.7k -> 1k; footprint _0603-W -> _std:_0603-W; moved to F.Cu
- R12, R13: value 22 -> 4.7k; footprint _0603-W -> _std:_0603-W
- R3, R4: value R -> 10k; footprint _0603-W -> _std:_0603-W
- R6, R7, R8: value 1k -> 10k; footprint _0603-W -> _std:_0603-W; moved to F.Cu
- R9: value 1k -> 100k; footprint _0603-W -> _std:_0603-W; moved to F.Cu
- U1: value 24LC128 -> STM32F042C6T6; footprint _TSSOP-8 -> _lqfp:_LQFP48; moved to F.Cu
- U2: value STM32F415RGT6 -> MIC5201-3.3YS; footprint _LQFP64 -> _std:_SOT23-3
- U3: value LTC4412 -> H3LIS331DL; footprint _TSOT23-6 -> _sensors:_H3LIS331DL; moved to F.Cu
- U4: value MAX3051 -> MPU6000; footprint _SOT23-8 -> _sensors:_MPU-60X0; moved to F.Cu
- U5: value LT1965 -> MS5611-01BA; footprint _MSOP-8-EP -> _sensors:_MS5611-01BA
- X1: footprint _TSX-3225-SMD-XTAL -> _div:_TSX-3225-SMD-XTAL
- moved R3 119.8 mm to (151.3, 58.6), turned to 0 degrees
- moved U5 116.3 mm to (153.0, 53.9)
- moved P2 114.6 mm to (145.5, 54.9), turned to 0 degrees
- moved C17 114.1 mm to (151.3, 57.0), turned to 0 degrees
- moved R4 111.3 mm to (153.9, 57.0)
- moved C20 111.3 mm to (143.8, 62.7), turned to 0 degrees
- moved R13 107.3 mm to (152.0, 63.7), turned to 0 degrees
- moved C13 106.7 mm to (146.7, 69.6), turned to 0 degrees
- moved R6 106.6 mm to (139.0, 71.1), turned to 0 degrees
- moved C18 106.3 mm to (148.7, 59.0), turned to 0 degrees
- moved R11 103.9 mm to (146.9, 67.4), turned to 0 degrees
- moved R12 103.1 mm to (149.4, 65.2)
- moved R2 100.6 mm to (148.7, 60.6), turned to 0 degrees
- moved C16 100.4 mm to (153.8, 58.6)
- moved R10 99.6 mm to (141.6, 71.1), turned to 0 degrees
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Connections:
- C1 pad 1: N-0000078 -> VCC
- C10 pad 1: VCC -> Net-(C10-Pad1)
- C11 pad 1: N-000004 -> Net-(C11-Pad1)
- C12 pad 1: N-000005 -> /V_DC
- C13 pad 1: /Sensors/VCC_A -> VCC
- C15 pad 1: N-0000048 -> VCC
- C16 pad 1: N-0000047 -> VCC
- C17 pad 1: /V_DC -> GND
- C17 pad 2: GND -> Net-(C17-Pad2)
- C18 pad 1: /V_IN -> VCC
- C19 pad 1: VCC -> Net-(C19-Pad1)
- C2 pad 1: VCC -> /V_BAT_MON_AD
- C20 pad 1: /V_DC -> VCC
- C21 pad 1: N-0000060 -> VCC
- C3 pad 1: N-0000078 -> VCC
- C4 pad 1: /V_BAT_MON_AD -> VCC
- C8 pad 1: VCC -> /STM32F4_NRST
- CONN1 pad 4: /STM32F4_TRST -> /STM32F4_SWDIO
- CONN1 pad 5: /STM32F4_TDI -> /STM32F4_SWCLK
- CONN2 pad 1: /SDIO_D2 -> Net-(CONN2-Pad1)
- CONN2 pad 2: /SDIO_D3 -> /SD_CS
- CONN2 pad 3: /SDIO_CMD -> /SD_DIN
- CONN2 pad 4: N-0000078 -> VCC
- CONN2 pad 5: /SDIO_CK -> /SD_CLK
- CONN2 pad 7: /SDIO_D0 -> /SD_DOUT
- CONN2 pad 8: /SDIO_D1 -> Net-(CONN2-Pad8)
- CONN3 pad 1: /V_USB -> VCC
- CONN3 pad 2: N-0000044 -> GND
- CONN3 pad 3: N-0000045 -> /UART_TX
- CONN3 pad 4: (no net) -> /UART_RX
- D1 pad 1: N-0000054 -> /ERROR_LED
- D1 pad 2: GND -> Net-(D1-Pad2)
- D2 pad 1: N-0000011 -> /HEARTBEAT_LED
- D2 pad 2: GND -> Net-(D2-Pad2)
- P1 pad 1: /V_DC -> VCC
- R1 pad 1: /SD_LED -> /V_BAT_MON_AD
- R1 pad 2: N-0000054 -> /V_DC
- R10 pad 1: /Sensors/VCC_A -> Net-(D1-Pad2)
- R10 pad 2: /Sensors/I2C_SCL -> GND
- R11 pad 1: /Sensors/VCC_A -> Net-(D2-Pad2)
- R11 pad 2: /Sensors/I2C_SDA -> GND
- R12 pad 1: N-0000044 -> VCC
- R12 pad 2: /USB_DM -> /INT_I2C_SCL
- R13 pad 1: /USB_DP -> VCC
- R13 pad 2: N-0000045 -> /INT_I2C_SDA
- R2 pad 1: VCC -> /V_BAT_MON_AD
- R2 pad 2: /SD_PWR -> GND
- R3 pad 1: /V_BAT_MON_AD -> VCC
- R3 pad 2: /V_DC -> Net-(CONN2-Pad8)
- R4 pad 1: /V_BAT_MON_AD -> VCC
- R4 pad 2: GND -> /SD_DOUT
- R5 pad 1: /STM32F4_NRST -> VCC
- R5 pad 2: VCC -> /SD_CLK
- R6 pad 2: N-0000011 -> /SD_DIN
- R7 pad 1: N-0000050 -> VCC
- R7 pad 2: GND -> /SD_CS
- R8 pad 1: N-0000039 -> VCC
- R8 pad 2: GND -> Net-(CONN2-Pad1)
- R9 pad 1: N-0000034 -> /STM32F4_NRST
- R9 pad 2: GND -> VCC
- U1 pad 1: GND -> VCC
- U1 pad 2: GND -> Net-(U1-Pad2)
- U1 pad 3: GND -> Net-(U1-Pad3)
- U1 pad 4: GND -> Net-(U1-Pad4)
- U1 pad 5: /Sensors/I2C_SDA -> Net-(C10-Pad1)
- U1 pad 6: /Sensors/I2C_SCL -> Net-(C11-Pad1)
- U1 pad 7: GND -> /STM32F4_NRST
- U1 pad 8: /Sensors/VCC_A -> GND
- U2 pad 1: VCC -> /V_DC
- U2 pad 2: /SD_PWR -> GND
- U2 pad 3: /EN_VCC_A -> VCC
- U3 pad 1: /V_DC -> VCC
- U3 pad 2: GND -> (no net)
- U3 pad 3: GND -> (no net)
- U3 pad 4: (no net) -> /INT_I2C_SCL
- U3 pad 5: N-0000051 -> GND
- U3 pad 6: /V_IN -> /INT_I2C_SDA
- U4 pad 1: /CAN_CONN1_TX -> GND
- U4 pad 2: GND -> (no net)
- U4 pad 3: VCC -> (no net)
- U4 pad 4: /CAN_CONN1_RX -> (no net)
- U4 pad 5: GND -> (no net)
- U4 pad 8: N-000003 -> VCC
- U5 pad 1: /VCC_IO -> VCC
- U5 pad 2: /VCC_IO -> VCC
- U5 pad 3: /VCC_IO -> GND
- U5 pad 6: /IO_EN -> Net-(U5-Pad6)
- U5 pad 7: /V_DC -> /INT_I2C_SDA
- U5 pad 8: /V_DC -> /INT_I2C_SCL
- X1 pad 1: N-0000047 -> Net-(C11-Pad1)
- X1 pad 3: N-0000048 -> Net-(C10-Pad1)
Routing:
- net GND: track 149.3 -> 0.00 mm, vias 26 -> 0
- net /VCC_IO: track 96.5 -> 0.00 mm, vias 5 -> 0
- net VCC: track 81.5 -> 0.00 mm, vias 8 -> 0
- net /V_BAT_MON_AD: track 56.6 -> 0.00 mm, vias 4 -> 0
- net /IO_EN: track 51.3 -> 0.00 mm, vias 3 -> 0
- net /Sensors/VCC_A: track 43.6 -> 0.00 mm, vias 5 -> 0
- net /I2C_CONN1_SDA: track 43.2 -> 0.00 mm, vias 2 -> 0
- net /I2C_CONN1_SCL: track 40.5 -> 0.00 mm, vias 2 -> 0
- net /Sensors/I2C_SDA: track 35.3 -> 0.00 mm, vias 5 -> 0
- net /STM32F4_NRST: track 35.1 -> 0.00 mm, vias 2 -> 0
- net /Sensors/I2C_SCL: track 34.3 -> 0.00 mm, vias 3 -> 0
- net Net-(U4-Pad6): track 32.7 -> 0.00 mm
- net Net-(U4-Pad7): track 32.4 -> 0.00 mm
- net /V_USB: track 27.2 -> 0.00 mm, vias 2 -> 0
- net /V_DC: track 27.1 -> 0.00 mm, vias 1 -> 0
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- removed copper zone on Inner2.Cu, net /Sensors/VCC_A
- removed copper zone on B.Cu, net GND
- removed copper zone on F.Cu, net GND
- removed copper zone on Inner1.Cu(GND), net GND
- removed copper zone on Inner2.Cu, net GND
- removed copper zone on Inner2.Cu, net VCC
Other:
- board outline removed
- copper layers 4 -> 2
- net class Default: clearance 0.2032 -> 0.2; trace_width 0.2032 -> 0.25; via_dia 0.706 -> 1; via_drill 0.3 -> 0.5
- rule trace_clearance: 0.2032 -> 0.2
- rule trace_min: 0.1524 -> 0.2
- rule via_min_size: 0.706 -> 0.4
- board text removed: "+"
- board text removed: "Board Dimension: 50mm x 23mm"
- board text removed: "CAN"
- board text removed: "I2C"
- board text removed: "PWR"
- board text removed: "REV A"
- board text removed: "UART1"
- board text removed: "UART2"
- board text removed: "UART3"
- board text removed: "UART4"
- board text removed: "Via Sizes: drill: 0.3mm diam: 0.706mm Track Size: 8mil = 0.203mm minimal spacing: 8mil"
